Commit message: fixes for mapping and sending templates to execution

File: Actuation/panda_ros/urdfs/panda.urdf (robot description, URDF)
Before this commit: robot panda_kinect, 17 links, 16 joints
Links:
- added link map
Joints:
- added joint panda_base_map: type fixed, parent panda_link0, child map, origin xyz=0 0 0.0 rpy=0 0 0, axis 0 0 0

Commit message: start of FT node code

File: Actuation/panda_ros/urdfs/panda.urdf (robot description, URDF)
Before this commit: robot panda_kinect, 18 links, 17 joints
Links:
- added link panda_orbital
Joints:
- added joint panda_orbital_joint: type fixed, parent panda_link8, child panda_orbital, origin xyz=-0.000 -0.000 0.144 rpy=3.1416 0.000 -0.785, axis 0 0 0
