Commit message: additional small fixes and compile scripts

File: ULIConfig/urdfs/panda.urdf (robot description, URDF)
Before this commit: robot panda_kinect, 18 links, 17 joints
Joints:
- joint fake_base: origin xyz=0.08211274 0.0 0.00823 rpy=3.14 -1.57 0.0 -> xyz=0.08211274 0.0 0.02823 rpy=3.14 -1.57 0.0
