Commit message: force torque sensor related

File: Actuation/config/panda.urdf (robot description, URDF)
Before this commit: robot panda_kinect, 19 links, 18 joints
Links:
- removed link sander
- added link ft_sensor_mid_link
- added link panda_orbital
- added link panda_orbital_COM
- link camera_body: geometry visual mesh filename=package://uli_config/meshes/visual/kinect-model.stl
- link ft_sensor_link: geometry collision mesh filename=package://uli_config/meshes/force_torque_sensor.stl; visual mesh filename=package://uli_config/meshes/force_torque_sensor.dae
- link panda_hand: geometry collision mesh filename=package://franka_description/meshes/collision/hand.stl; visual mesh filename=package://franka_description/meshes/visual/hand.dae
- link panda_leftfinger: geometry collision mesh filename=package://franka_description/meshes/collision/finger.stl; visual mesh filename=package://franka_description/meshes/visual/finger.dae
- link panda_link0: geometry collision mesh filename=package://franka_description/meshes/collision/link0.stl; visual mesh filename=package://franka_description/meshes/visual/link0.dae
- link panda_link1: geometry collision mesh filename=package://franka_description/meshes/collision/link1.stl; visual mesh filename=package://franka_description/meshes/visual/link1.dae
- link panda_link2: geometry collision mesh filename=package://franka_description/meshes/collision/link2.stl; visual mesh filename=package://franka_description/meshes/visual/link2.dae
- link panda_link3: geometry collision mesh filename=package://franka_description/meshes/collision/link3.stl; visual mesh filename=package://franka_description/meshes/visual/link3.dae
- link panda_link4: geometry collision mesh filename=package://franka_description/meshes/collision/link4.stl; visual mesh filename=package://franka_description/meshes/visual/link4.dae
- link panda_link5: geometry collision mesh filename=package://franka_description/meshes/collision/link5.stl; visual mesh filename=package://franka_description/meshes/visual/link5.dae
- link panda_link6: geometry collision mesh filename=package://franka_description/meshes/collision/link6.stl; visual mesh filename=package://franka_description/meshes/visual/link6.dae
- link panda_link7: geometry collision mesh filename=package://franka_description/meshes/collision/link7.stl; visual mesh filename=package://franka_description/meshes/visual/link7.dae
- link panda_rightfinger: geometry collision mesh filename=package://franka_description/meshes/collision/finger.stl; visual mesh filename=package://franka_description/meshes/visual/finger.dae
Joints:
- removed joint sander_joint
- added joint ft_mid_sensor_joint: type fixed, parent panda_link8, child ft_sensor_mid_link, origin xyz=0 0 0.0464 rpy=0 0 1.8326, axis 0 0 0
- added joint panda_orbital_COM_joint: type fixed, parent ft_sensor_link, child panda_orbital_COM, origin xyz=-0.000 -0.000 0.072 rpy=3.1416 0.000 -0.785, axis 0 0 0
- added joint panda_orbital_joint: type fixed, parent ft_sensor_link, child panda_orbital, origin xyz=-0.000 -0.000 0.144 rpy=3.1416 0.000 -0.785, axis 0 0 0
- joint fake_base: origin xyz=0.08211274 0.0 0.00823 rpy=3.14 -1.57 0.0 -> xyz=0.08211274 0.0 0.02823 rpy=3.14 -1.57 0.0
- joint ft_sensor_joint: origin xyz=0 0 0.062 rpy=0 0 0 -> xyz=0 0 0.06534 rpy=0 0 0; parent panda_link7 -> panda_link8
- joint panda_joint4: limit lower=-3.0718 upper=-0.3698 effort=87 velocity=2.1750 -> lower=-3.0718 upper=-0.0698 effort=87 velocity=2.1750
- joint panda_joint8: origin xyz=0 0 0.11 rpy=0 0 0 -> xyz=0 0 0.107 rpy=0 0 0; parent ft_sensor_link -> panda_link7

Commit message: fix FT in urdf

File: Actuation/config/panda.urdf (robot description, URDF)
Before this commit: robot panda_kinect, 21 links, 20 joints
Joints:
- joint panda_hand_joint: parent panda_link8 -> ft_sensor_link

Commit message: many fixes for panda sim

File: Actuation/config/panda.urdf (robot description, URDF)
Before this commit: robot panda_kinect, 21 links, 20 joints
Links:
- link camera_body: geometry visual mesh filename=package://panda_sim/meshes/visual/kinect-model.stl
- link ft_sensor_link: geometry collision mesh filename=package://panda_sim/meshes/force_torque_sensor.stl; visual mesh filename=package://panda_sim/meshes/force_torque_sensor.dae
- link panda_leftfinger: geometry visual mesh filename=package://franka_description/meshes/visual/finger.dae
- link panda_rightfinger: geometry visual mesh filename=package://franka_description/meshes/visual/finger.dae

Commit message: new surface model for IRC piece, sim fixes, and urdf updates for visual:

File: Actuation/config/panda.urdf (robot description, URDF)
Before this commit: robot panda_kinect, 21 links, 20 joints
Links:
- removed link panda_gripper
- removed link panda_hand
- removed link panda_leftfinger
- removed link panda_rightfinger
- added link panda_flange
- link panda_orbital: geometry visual mesh filename=package://panda_sim/meshes/sander_orbital_w_vib.STL
Joints:
- removed joint panda_finger_joint1
- removed joint panda_finger_joint2
- removed joint panda_gripper_joint
- removed joint panda_hand_joint
- added joint panda_flange_rotated_joint: type fixed, parent ft_sensor_link, child panda_flange, origin xyz=0 0 0 rpy=0 0 -0.785398163397
- joint fake_base: parent panda_hand -> panda_flange

Commit message: start of panda urdf camera fixes

File: Actuation/config/panda.urdf (robot description, URDF)
Before this commit: robot panda_kinect, 18 links, 17 joints
Links:
- added link camera_basenonrotated
- added link camera_holder; visual mesh filename=package://panda_sim/meshes/camera_holder_assem.STL
- added link panda_flange_original
Joints:
- added joint camera_holder_joint: type fixed, parent panda_flange_original, child camera_holder, origin xyz=0 0 0.0114808 rpy=3.14 0.0 0.0
- added joint camera_rotation: type fixed, parent camera_basenonrotated, child camera_base, origin xyz=0.0 0.0 0.0 rpy=0 -0.16069 0
- added joint panda_flange_original_joint: type fixed, parent panda_link8, child panda_flange_original, origin xyz=0 0 0 rpy=0 0 -0.785398163397
- joint fake_base: child camera_base -> camera_basenonrotated; origin xyz=0.08211274 0.0 0.02823 rpy=3.14 -1.57 0.0 -> xyz=0.093997 0.0 0.0266868 rpy=3.14 -1.57 0.0; parent panda_flange -> panda_flange_original

Commit message: stashed changes 5-9-22

File: Actuation/config/panda.urdf (robot description, URDF)
Before this commit: robot panda_kinect, 18 links, 17 joints
Links:
- added link camera_basenonrotated
- added link camera_holder; visual mesh filename=package://panda_sim/meshes/camera_holder_assem.STL
- added link camera_tripod
- added link panda_flange_original
Joints:
- added joint camera_holder_joint: type fixed, parent panda_flange_original, child camera_holder, origin xyz=0 0 0.0114808 rpy=3.14 0.0 0.0
- added joint camera_rotation: type fixed, parent camera_basenonrotated, child camera_tripod, origin xyz=0.0 0.0 0.0 rpy=0 -0.16069 0
- added joint camera_tripod_joint: type fixed, parent camera_tripod, child camera_base, origin xyz=0.062 0.0 0.0068 rpy=0 0 0
- added joint panda_flange_original_joint: type fixed, parent panda_link8, child panda_flange_original, origin xyz=0 0 0 rpy=0 0 -0.785398163397
- joint fake_base: child camera_base -> camera_basenonrotated; origin xyz=0.08211274 0.0 0.02823 rpy=3.14 -1.57 0.0 -> xyz=0.093997 0.0 0.0266868 rpy=3.14 -1.57 0.0; parent panda_flange -> panda_flange_original
